Commit message: fix error of section6.2.3

File: ROS_YuXiang/test6.2_make_robot/src/fishbot_description/urdf/first_robot.urdf.xacro (robot description, xacro)
@@ -7,8 +7,8 @@
                 <origin rpy="0 0 0" xyz="0 0 0"/>
                 <geometry>
-                    <cylinder length="${length}" radius="${radius}"/>
+                    <cylinder radius="${radius}" length="${length}"/>
                 </geometry>
-                <material name="red">
-                    <color rgba="1.0 0.0 0.0 1.0"/>
+                <material name="yellow">
+                    <color rgba="1.0 1.0 0.0 1.0"/>
                 </material>
             </visual>
@@ -23,8 +23,8 @@
                     <box size="0.02 0.02 0.02"/>
                 </geometry>
+                <material name="blue">
+                    <color rgba="0.0 0.0 1.0 1.0"/>
+                </material>
             </visual>
-            <material name="blue">
-                <color rgba="0.0 0.0 1.0 1.0"/>
-            </material>
         </link>
         <joint name="${imu_name}_joint" type="fixed">
