Commit message: fix robot geometry

File: ROS_YuXiang/test6.2_make_robot/src/fishbot_description/urdf/fishbot/base.urdf.xacro (robot description, xacro)
@@ -8,6 +8,6 @@
                     <cylinder radius="${radius}" length="${length}"/>
                 </geometry>
-                <material name="Grey">
-                    <color rgba="0.5 0.5 0.5 1.0"/>
+                <material name="white">
+                    <color rgba="1.0 1.0 1.0 0.5"/>
                 </material>
             </visual>

File: ROS_YuXiang/test6.2_make_robot/src/fishbot_description/urdf/fishbot/sensor/camera.urdf.xacro (robot description, xacro)
@@ -9,6 +9,6 @@
                     <box size="0.02 0.10 0.02"/>
                 </geometry>
-                <material name="Grey">
-                    <color rgba="0.5 0.5 0.5 1"/>
+                <material name="red">
+                    <color rgba="1.0 0.0 0.0 1.0"/>
                 </material>
             </visual>

File: ROS_YuXiang/test6.2_make_robot/src/fishbot_description/urdf/fishbot/sensor/imu.urdf.xacro (robot description, xacro)
@@ -8,6 +8,6 @@
                     <box size="0.02 0.02 0.02"/>
                 </geometry>
-                <material name="Grey">
-                    <color rgba="0.5 0.5 0.5 1.0"/>
+                <material name="black">
+                    <color rgba="0.0 0.0 0.0 0.8"/>
                 </material>
             </visual>

File: ROS_YuXiang/test6.2_make_robot/src/fishbot_description/urdf/fishbot/sensor/laser.urdf.xacro (robot description, xacro)
@@ -7,8 +7,8 @@
                 <origin xyz="0 0 0" rpy="0 0 0"/>
                 <geometry>
-                    <cylinder radius="0.10" length="0.01"/>
+                    <cylinder radius="0.01" length="0.10"/>
                 </geometry>
-                <material name="white">
-                    <color rgba="1 1 1 1"/>
+                <material name="green">
+                    <color rgba="0.0 1.0 0.0 0.8"/>
                 </material>
             </visual>
@@ -26,6 +26,6 @@
                     <cylinder radius="0.02" length="0.02"/>
                 </geometry>
-                <material name="white">
-                    <color rgba="1 1 1 1"/>
+                <material name="green">
+                    <color rgba="0.0 1.0 0.0 0.8"/>
                 </material>
             </visual>

Commit message: section6.2.6, add ground, you need set fixed_frame into base_footprint in the RViz2

File: ROS_YuXiang/test6.2_make_robot/src/fishbot_description/urdf/fishbot/base.urdf.xacro (robot description, xacro)
@@ -13,4 +13,10 @@
             </visual>
         </link>
+        <link name="base_footprint" />
+        <joint name="base_joint" type="fixed">"
+            <parent link="base_footprint"/>
+            <child link="base_link"/>
+            <origin xyz="0 0 ${length/2.0+0.032-0.001}" rpy="0 0 0"/>
+        </joint>
     </xacro:macro>
 </robot>
