Commit message: fix error of actuator wheel

File: ROS_YuXiang/test6.2_make_robot/src/fishbot_description/urdf/fishbot/actuator/wheel.urdf.xacro (robot description, xacro)
@@ -4,5 +4,5 @@
         <link name="${wheel_name}_wheel_link">
             <visual>
-                <origin xyz="${xyz}" rpy="1.57079 0 0"/>
+                <origin xyz="0 0 0" rpy="1.57079 0 0"/>
                 <geometry>
                     <cylinder radius="0.032" length="0.04"/>

File: ROS_YuXiang/test6.2_make_robot/src/fishbot_description/urdf/fishbot/fishbot.urdf.xacro (robot description, xacro)
@@ -15,6 +15,6 @@
     <xacro:include filename="$(find fishbot_description)/urdf/fishbot/actuator/caster.urdf.xacro"/>
     <!-- 执行器主动轮 + 从动轮 -->
-    <xacro:wheel_xacro wheel_name="left" xyz="0.0 0.05 -0.06" />
-    <xacro:wheel_xacro wheel_name="right" xyz="0.0 -0.05 -0.06" />
+    <xacro:wheel_xacro wheel_name="left" xyz="0.0 0.10 -0.06" />
+    <xacro:wheel_xacro wheel_name="right" xyz="0.0 -0.10 -0.06" />
     <xacro:caster_xacro caster_name="front" xyz="0.08 0.0 -0.076" />
     <xacro:caster_xacro caster_name="back" xyz="-0.08 0.0 -0.076" />
