Commit message: section6.3.1, add collision

File: ROS_YuXiang/test6.2_make_robot/src/fishbot_description/urdf/fishbot/actuator/caster.urdf.xacro (robot description, xacro)
@@ -12,4 +12,13 @@
             </material>
         </visual>
+        <collision>
+            <origin xyz="0 0 0" rpy="0 0 0"/>
+            <geometry>
+                <sphere radius="0.016"/>
+            </geometry>
+            <material name="yellow">
+                <color rgba="1.0 1.0 0.0 1.0"/>
+            </material>
+        </collision>
         </link>
         <joint name="${caster_name}_caster_joint" type="fixed">

File: ROS_YuXiang/test6.2_make_robot/src/fishbot_description/urdf/fishbot/actuator/wheel.urdf.xacro (robot description, xacro)
@@ -12,4 +12,13 @@
                 </material>
             </visual>
+            <collision>
+                <origin xyz="0 0 0" rpy="1.57079 0 0"/>
+                <geometry>
+                    <cylinder radius="0.032" length="0.04"/>
+                </geometry>
+                <material name="yellow">
+                    <color rgba="1 1 0 0.8"/>
+                </material>
+            </collision>
         </link>
         <joint name="${wheel_name}_wheel_joint" type="continuous">

File: ROS_YuXiang/test6.2_make_robot/src/fishbot_description/urdf/fishbot/base.urdf.xacro (robot description, xacro)
@@ -12,4 +12,13 @@
                 </material>
             </visual>
+            <collision>
+                <origin rpy="0 0 0" xyz="0 0 0"/>
+                <geometry>
+                    <cylinder radius="${radius}" length="${length}"/>
+                </geometry>
+                <material name="white">
+                    <color rgba="1.0 1.0 1.0 0.5"/>
+                </material>
+            </collision>
         </link>
         <link name="base_footprint" />

File: ROS_YuXiang/test6.2_make_robot/src/fishbot_description/urdf/fishbot/sensor/camera.urdf.xacro (robot description, xacro)
@@ -13,4 +13,13 @@
                 </material>
             </visual>
+            <collision>
+                <origin xyz="0 0 0" rpy="0 0 0"/>
+                <geometry>
+                    <box size="0.02 0.10 0.02"/>
+                </geometry>
+                <material name="red">
+                    <color rgba="1.0 0.0 0.0 1.0"/>
+                </material>
+            </collision>
         </link>
         <joint name="camera_joint" type="fixed">

File: ROS_YuXiang/test6.2_make_robot/src/fishbot_description/urdf/fishbot/sensor/imu.urdf.xacro (robot description, xacro)
@@ -12,4 +12,13 @@
                 </material>
             </visual>
+            <collision>
+                <origin xyz="0 0 0" rpy="0 0 0"/>
+                <geometry>
+                    <box size="0.02 0.02 0.02"/>
+                </geometry>
+                <material name="black">
+                    <color rgba="0.0 0.0 0.0 0.8"/>
+                </material>
+            </collision>
         </link>
         <joint name="imu_joint" type="fixed">

File: ROS_YuXiang/test6.2_make_robot/src/fishbot_description/urdf/fishbot/sensor/laser.urdf.xacro (robot description, xacro)
@@ -13,4 +13,13 @@
                 </material>
             </visual>
+            <collision>
+                <origin xyz="0 0 0" rpy="0 0 0"/>
+                <geometry>
+                    <cylinder radius="0.01" length="0.10"/>
+                </geometry>
+                <material name="green">
+                    <color rgba="0.0 1.0 0.0 0.8"/>
+                </material>
+            </collision>
         </link>
         <joint name="laser_cylinder_joint" type="fixed">
@@ -30,4 +39,13 @@
                 </material>
             </visual>
+            <collision>
+                <origin xyz="0 0 0" rpy="0 0 0"/>
+                <geometry>
+                    <cylinder radius="0.02" length="0.02"/>
+                </geometry>
+                <material name="green">
+                    <color rgba="0.0 1.0 0.0 0.8"/>
+                </material>
+            </collision>
         </link>
         <joint name="laser_joint" type="fixed">

Commit message: section6.4.3, define color and friction of robot parts

File: ROS_YuXiang/test6.2_make_robot/src/fishbot_description/urdf/fishbot/actuator/caster.urdf.xacro (robot description, xacro)
@@ -3,4 +3,10 @@
     <xacro:include filename="$(find fishbot_description)/urdf/fishbot/common_inertia.xacro"/>
     <xacro:macro name="caster_xacro" params="caster_name xyz">
+        <gazebo reference="${caster_name}_caster_link">
+            <mu1 value="0.0"/>
+            <mu2 value="0.0"/>
+            <kp value="1000000000.0"/>
+            <kd value="1.0"/>
+        </gazebo>
         <link name="${caster_name}_caster_link">
         <visual>

File: ROS_YuXiang/test6.2_make_robot/src/fishbot_description/urdf/fishbot/actuator/wheel.urdf.xacro (robot description, xacro)
@@ -3,4 +3,11 @@
     <xacro:include filename="$(find fishbot_description)/urdf/fishbot/common_inertia.xacro"/>
     <xacro:macro name="wheel_xacro" params="wheel_name xyz">
+        <gazebo reference="${wheel_name}_wheel_link">
+            <!-- mu1:切向摩擦系数，mu2:法向摩擦系数，kp:接触刚度系数，kd:阻尼系数 -->
+            <mu1 value="20.0"/>
+            <mu2 value="20.0"/>
+            <kp value="1000000000.0"/>
+            <kd value="1.0"/>
+        </gazebo>
         <link name="${wheel_name}_wheel_link">
             <visual>

File: ROS_YuXiang/test6.2_make_robot/src/fishbot_description/urdf/fishbot/sensor/laser.urdf.xacro (robot description, xacro)
@@ -3,4 +3,10 @@
     <xacro:include filename="$(find fishbot_description)/urdf/fishbot/common_inertia.xacro"/>
     <xacro:macro name="laser_xacro" params="xyz">
+        <gazebo reference="laser_link">
+            <material>Gazebo/Black</material>
+        </gazebo>
+        <gazebo reference="laser_cylinder_link">
+            <material>Gazebo/Black</material>
+        </gazebo>
         <!-- ==========雷达支撑杆========== -->
         <link name="laser_cylinder_link">
